Commit message: 4th commit

File: motoman_move_glass/urdf/glass_panel.urdf.xacro (robot description, xacro)
@@ -18,7 +18,7 @@
                     <box size="0.4 1 0.005"/>
                 </geometry>
-  13            <material name="Cyan">
-  14                <color rgba="0 1.0 1.0 1.0"/>
-  15            </material>
+                <material name="Cyan">
+                    <color rgba="0 1.0 1.0 1.0"/>
+                </material>
             </visual>
             <collision>

File: motoman_move_glass/urdf/robots.urdf.xacro (robot description, xacro)
@@ -42,3 +42,4 @@
     <xacro:glass_panel parent="vacuum_gripper_top">
     </xacro:glass_panel>
+    <xacro:include filename="$(find motoman_move_glass)/urdf/common.xacro"/>
 </robot>
